Commit message: adding initial trr sim

File: urdf/sensors_gazebo.urdf.xacro (robot description, xacro)
@@ -4,5 +4,5 @@
     <gazebo reference="camera_link">
       <sensor type="camera" name="${cam_name}">
-	<update_rate>30.0</update_rate>
+	<update_rate>10.0</update_rate>
 	<camera name="head">
           <horizontal_fov>1.3962634</horizontal_fov>
@@ -42,3 +42,81 @@
     </gazebo>
   </xacro:macro>
+  <xacro:macro name="gazebo_rpi_camera" params="cam_name">
+    <gazebo reference="camera1_link">
+      <sensor type="camera" name="${cam_name}">
+	<update_rate>10.0</update_rate>
+	<camera name="head">
+          <horizontal_fov>2.3</horizontal_fov>   <!--<horizontal_fov>1.5</horizontal_fov>-->
+          <image>
+            <width>640</width>    <!--<width>1280</width>-->
+            <height>360</height>   <!--<height>720</height>-->
+            <format>R8G8B8</format>
+          </image>
+          <clip>
+            <near>0.02</near>
+            <far>50</far>
+          </clip>
+          <noise>
+            <type>gaussian</type>
+            <!-- Noise is sampled independently per pixel on each frame.
+		 That pixel's noise value is added to each of its color
+		 channels, which at that point lie in the range [0,1]. -->
+            <mean>0.0</mean>
+            <stddev>0.007</stddev>
+          </noise>
+	</camera>
+	<plugin name="camera_controller" filename="libgazebo_ros_camera.so">
+          <alwaysOn>true</alwaysOn>
+          <updateRate>0.0</updateRate>
+          <cameraName>${cam_name}</cameraName>
+          <imageTopicName>image_raw</imageTopicName>
+          <cameraInfoTopicName>camera_info</cameraInfoTopicName>
+          <frameName>camera_link</frameName>
+          <hackBaseline>0.07</hackBaseline>
+          <distortionK1>0.0</distortionK1>
+          <distortionK2>0.0</distortionK2>
+          <distortionK3>0.0</distortionK3>
+          <distortionT1>0.0</distortionT1>
+          <distortionT2>0.0</distortionT2>
+	</plugin>
+      </sensor>
+    </gazebo>
+  </xacro:macro>
+  <xacro:macro name="gazebo_hokuyo" params="laser_name">
+    <gazebo reference="hokuyo_link">
+    <sensor type="gpu_ray" name="head_hokuyo_sensor">
+      <pose>0 0 0 0 0 0</pose>
+      <visualize>false</visualize>
+      <update_rate>40</update_rate>
+      <ray>
+        <scan>
+          <horizontal>
+            <samples>1080</samples>
+            <resolution>0.25</resolution>
+            <min_angle>-2.3561945</min_angle>
+            <max_angle>2.3561945</max_angle>
+          </horizontal>
+        </scan>
+        <range>
+          <min>0.10</min>
+          <max>30.0</max>
+          <resolution>0.01</resolution>
+        </range>
+        <noise>
+          <type>gaussian</type>
+          <!-- Noise parameters based on published spec for Hokuyo laser
+               achieving "+-30mm" accuracy at range < 10m.  A mean of 0.0m and
+               stddev of 0.01m will put 99.7% of samples within 0.03m of the true
+               reading. -->
+          <mean>0.0</mean>
+          <stddev>0.01</stddev>
+        </noise>
+      </ray>
+      <plugin name="gazebo_ros_head_hokuyo_controller" filename="libgazebo_ros_gpu_laser.so">
+        <topicName>laserscan</topicName>
+        <frameName>hokuyo_link</frameName>
+      </plugin>
+    </sensor>
+  </gazebo>
+  </xacro:macro>
 </robot>

Commit message: start_finish

File: urdf/sensors_gazebo.urdf.xacro (robot description, xacro)
@@ -83,4 +83,45 @@
     </gazebo>
   </xacro:macro>
+   <xacro:macro name="gazebo_ueye_camera" params="cam_name">
+    <gazebo reference="${cam_name}_link">
+      <sensor type="camera" name="${cam_name}">
+	<update_rate>10.0</update_rate>
+	<camera name="head">
+          <horizontal_fov>1.6</horizontal_fov>   <!--<horizontal_fov>1.5</horizontal_fov>-->
+          <image>
+            <width>752</width>    <!--<width>1280</width>-->
+            <height>480</height>   <!--<height>720</height>-->
+            <format>B8G8R8</format>
+          </image>
+          <clip>
+            <near>0.02</near>
+            <far>50</far>
+          </clip>
+          <noise>
+            <type>gaussian</type>
+            <!-- Noise is sampled independently per pixel on each frame.
+		 That pixel's noise value is added to each of its color
+		 channels, which at that point lie in the range [0,1]. -->
+            <mean>0.0</mean>
+            <stddev>0.007</stddev>
+          </noise>
+	</camera>
+	<plugin name="camera_controller" filename="libgazebo_ros_camera.so">
+          <alwaysOn>true</alwaysOn>
+          <updateRate>0.0</updateRate>
+          <cameraName>${cam_name}</cameraName>
+          <imageTopicName>image_raw</imageTopicName>
+          <cameraInfoTopicName>camera_info</cameraInfoTopicName>
+          <frameName>camera_link</frameName>
+          <hackBaseline>0.07</hackBaseline>
+          <distortionK1>0.0</distortionK1>
+          <distortionK2>0.0</distortionK2>
+          <distortionK3>0.0</distortionK3>
+          <distortionT1>0.0</distortionT1>
+          <distortionT2>0.0</distortionT2>
+	</plugin>
+      </sensor>
+    </gazebo>
+  </xacro:macro>
   <xacro:macro name="gazebo_hokuyo" params="laser_name">
     <gazebo reference="hokuyo_link">

Commit message: bla

File: urdf/sensors_gazebo.urdf.xacro (robot description, xacro)
@@ -141,5 +141,5 @@
         <range>
           <min>0.10</min>
-          <max>30.0</max>
+          <max>16.0</max>
           <resolution>0.01</resolution>
         </range>
@@ -161,3 +161,37 @@
   </gazebo>
   </xacro:macro>
+  <xacro:macro name="gazebo_rplidar" params="laser_name">
+    <gazebo reference="hokuyo_link">
+    <sensor type="ray" name="head_hokuyo_sensor"> <!-- gpu_ray ?? -->
+      <pose>0 0 0 0 0 0</pose>
+      <visualize>false</visualize>
+      <update_rate>5</update_rate>
+      <ray>
+        <scan>
+          <horizontal>
+            <samples>360</samples>
+            <resolution>1.</resolution>
+            <min_angle>0</min_angle>
+            <max_angle>6.28319</max_angle>
+          </horizontal>
+        </scan>
+        <range>
+          <min>0.12</min>
+          <max>3.5</max>
+          <resolution>0.01</resolution>
+        </range>
+        <noise>
+          <type>gaussian</type>
+          <mean>0.0</mean>
+          <stddev>0.01</stddev>
+        </noise>
+      </ray>
+      <!-- <plugin name="gazebo_ros_head_hokuyo_controller" filename="libgazebo_ros_gpu_laser.so"> -->
+      <plugin name="gazebo_ros_head_hokuyo_controller" filename="libgazebo_ros_laser.so">
+        <topicName>laserscan</topicName>
+        <frameName>hokuyo_link</frameName>
+      </plugin>
+    </sensor>
+  </gazebo>
+  </xacro:macro>
 </robot>
